File: hw/pcbs/kbd.kicad_pcb (KiCad board)
At the start: 2 copper layers, 291.8 x 81 mm, 154 parts

Commit message: feat: add new kicad project
Parts:
- removed the ? at (234.4, 101.5)
- removed the ? at (234.4, 82.5)
- removed MCU2: Seeeduino XIAO-nrf52840, Seeeduino XIAO-MOUDLE14P-2.54-21X17.8MM
- removed the REF** at (171.1, 79.2)
- removed the REF** at (278.4, 97.0)
- removed the REF** at (135.5, 49.0)
- removed the REF** at (232.4, 98.6)
- removed the REF** at (299.7, 79.2)
- removed the REF** at (171.1, 61.5)
- removed the REF** at (296.1, 97.0)
- removed the REF** at (281.9, 43.7)
- removed the REF** at (370.8, 61.5)
- removed the REF** at (188.8, 43.7)
- removed the REF** at (322.8, 96.1)
- removed the REF** at (353.0, 61.5)
- removed the REF** at (135.5, 66.8)
- removed the REF** at (153.3, 57.9)
- removed the REF** at (353.0, 97.0)
- removed the REF** at (210.2, 97.0)
- removed the REF** at (317.5, 75.7)
- removed the REF** at (148.0, 93.3)
- removed the REF** at (317.5, 57.9)
- removed the REF** at (238.4, 98.6)
- removed the REF** at (117.8, 61.5)
- removed the REF** at (370.8, 97.0)
- removed the REF** at (192.4, 97.0)
- removed the REF** at (100.0, 61.5)
- removed the REF** at (188.8, 61.5)
- removed the REF** at (353.0, 79.2)
- removed the REF** at (153.3, 40.1)
- removed the REF** at (238.4, 101.4)
- removed the REF** at (335.2, 84.6)
- removed the REF** at (100.0, 97.0)
- removed the REF** at (281.9, 61.5)
- removed the REF** at (117.8, 97.0)
- removed the REF** at (370.8, 79.2)
- removed the REF** at (232.4, 101.4)
- removed the REF** at (171.1, 43.7)
- removed the REF** at (260.6, 97.0)
- removed the REF** at (117.8, 79.2)
- removed the REF** at (114.2, 50.2)
- removed the REF** at (153.3, 75.7)
- removed the REF** at (356.6, 50.2)
- removed the REF** at (299.7, 43.7)
- removed the REF** at (100.0, 79.2)
- removed the REF** at (188.8, 79.2)
- removed the REF** at (174.6, 97.0)
- removed the REF** at (281.9, 79.2)
- removed the REF** at (299.7, 61.5)
- removed the REF** at (335.2, 66.8)
- removed the REF** at (322.8, 93.3)
- removed the REF** at (317.5, 40.1)
- removed the REF** at (135.5, 84.6)
- removed the REF** at (335.2, 49.0)
- removed the REF** at (148.0, 96.1)
- removed _63, _64, _65, _66, _67, _68, _69, _70, _71, _72: , Mount_Hole_2.2mm_Pad_Via
- removed _73, _74, _75, _76: , Magnet_Hole_12.3mm
- added ?: , PAD-1.0922mm, F.Cu at (162.4, 154.0)
- added ?: , PAD-1.0922mm, F.Cu at (194.2, 143.8)
- added ?: , PAD-1.0922mm, F.Cu at (168.2, 139.9)
- added ?: , PAD-1.0922mm, F.Cu at (198.2, 143.8)
- added ?: , PAD-1.0922mm, F.Cu at (161.5, 156.3)
- added ?: , PAD-1.0922mm, F.Cu at (207.2, 142.3)
- added ?: , PAD-1.0922mm, F.Cu at (164.3, 149.3)
- added ?: , PAD-1.0922mm, F.Cu at (185.2, 137.2)
- added ?: , PAD-1.0922mm, F.Cu at (225.1, 142.2)
- added ?: , PAD-1.0922mm, F.Cu at (163.4, 151.6)
- added ?: , PAD-1.0922mm, F.Cu at (185.2, 144.8)
- added ?: , PAD-1.0922mm, F.Cu at (228.0, 149.3)
- added ?: , PAD-1.0922mm, F.Cu at (185.2, 132.1)
- added ?: , PAD-1.0922mm, F.Cu at (207.2, 129.6)
- added ?: , PAD-1.0922mm, F.Cu at (207.2, 124.5)
- added ?: , PAD-1.0922mm, F.Cu at (185.2, 124.5)
- added ?: , PAD-1.0922mm, F.Cu at (185.2, 139.8)
- added ?: , PAD-1.0922mm, F.Cu at (167.2, 142.2)
- added ?: , PAD-1.0922mm, F.Cu at (185.2, 122.0)
- added ?: , PAD-1.0922mm, F.Cu at (185.2, 142.3)
- added ?: , PAD-1.0922mm, F.Cu at (165.3, 146.9)
- added ?: , PAD-1.0922mm, F.Cu at (229.9, 154.0)
- added ?: , PAD-1.0922mm, F.Cu at (207.2, 127.1)
- added ?: , PAD-1.0922mm, F.Cu at (160.5, 158.7)
- added ?: , PAD-1.0922mm, F.Cu at (229.0, 151.6)
- added ?: , PAD-1.0922mm, F.Cu at (185.2, 134.7)
- added ?: , PAD-1.0922mm, F.Cu at (207.2, 122.0)
- added ?: , PAD-1.0922mm, F.Cu at (207.2, 137.2)
- added ?: , PAD-1.0922mm, F.Cu at (230.9, 156.3)
- added ?: , PAD-1.0922mm, F.Cu at (227.1, 146.9)
- added ?: , PAD-1.0922mm, F.Cu at (231.8, 158.7)
- added ?: , PAD-1.0922mm, F.Cu at (207.2, 144.8)
- added ?: , PAD-1.0922mm, F.Cu at (224.2, 139.9)
- added ?: , PAD-1.0922mm, F.Cu at (226.1, 144.6)
- added ?: , PAD-1.0922mm, F.Cu at (207.2, 134.7)
- added ?: , PAD-1.0922mm, F.Cu at (223.2, 137.5)
- added ?: , PAD-1.0922mm, F.Cu at (185.2, 127.1)
- added ?: , PAD-1.0922mm, F.Cu at (185.2, 129.6)
- added ?: , PAD-1.0922mm, F.Cu at (207.2, 139.8)
- added ?: , PAD-1.0922mm, F.Cu at (169.1, 137.5)
- added ?: , PAD-1.0922mm, F.Cu at (166.3, 144.6)
- added ?: , PAD-1.0922mm, F.Cu at (207.2, 132.1)
- added PWR1: , ceoloide:power_switch_smd_side, F.Cu at (196.2, 178.5)
- added REF**: VIA-0.6mm, VIA-0.6mm, F.Cu at (251.8, 152.3)
- added REF**: VIA-0.6mm, VIA-0.6mm, F.Cu at (237.6, 117.1)
- added REF**: VIA-0.6mm, VIA-0.6mm, F.Cu at (137.0, 171.4)
- added REF**: VIA-0.6mm, VIA-0.6mm, F.Cu at (269.4, 145.2)
- added REF**: VIA-0.6mm, VIA-0.6mm, F.Cu at (85.6, 136.3)
- added REF**: VIA-0.6mm, VIA-0.6mm, F.Cu at (121.0, 99.4)
- added REF**: VIA-0.6mm, VIA-0.6mm, F.Cu at (119.4, 164.3)
- added REF**: VIA-0.6mm, VIA-0.6mm, F.Cu at (237.8, 178.5)
- added REF**: VIA-0.6mm, VIA-0.6mm, F.Cu at (113.9, 117.0)
- added REF**: VIA-0.6mm, VIA-0.6mm, F.Cu at (273.0, 164.3)
- added REF**: VIA-0.6mm, VIA-0.6mm, F.Cu at (63.0, 141.5)
- added REF**: VIA-0.6mm, VIA-0.6mm, F.Cu at (322.3, 123.9)
- added REF**: VIA-0.6mm, VIA-0.6mm, F.Cu at (244.7, 134.7)
- added REF**: VIA-0.6mm, VIA-0.6mm, F.Cu at (262.3, 127.6)
- added REF**: VIA-0.6mm, VIA-0.6mm, F.Cu at (332.8, 99.1)
- added REF**: VIA-0.6mm, VIA-0.6mm, F.Cu at (77.2, 106.3)
- added REF**: VIA-0.6mm, VIA-0.6mm, F.Cu at (255.4, 171.4)
- added REF**: VIA-0.6mm, VIA-0.6mm, F.Cu at (70.1, 123.9)
- added REF**: VIA-0.6mm, VIA-0.6mm, F.Cu at (285.6, 134.6)
- added REF**: VIA-0.6mm, VIA-0.6mm, F.Cu at (306.8, 136.3)
- added REF**: VIA-0.6mm, VIA-0.6mm, F.Cu at (329.4, 141.5)
- added REF**: VIA-0.6mm, VIA-0.6mm, F.Cu at (339.9, 116.8)
- added REF**: VIA-0.6mm, VIA-0.6mm, F.Cu at (292.5, 101.0)
- added REF**: VIA-0.6mm, VIA-0.6mm, F.Cu at (147.7, 134.7)
- added REF**: VIA-0.6mm, VIA-0.6mm, F.Cu at (154.8, 117.1)
- added REF**: VIA-0.6mm, VIA-0.6mm, F.Cu at (130.1, 127.6)
- added REF**: VIA-0.6mm, VIA-0.6mm, F.Cu at (154.6, 178.5)
- added REF**: VIA-0.6mm, VIA-0.6mm, F.Cu at (278.5, 117.0)
- added REF**: VIA-0.6mm, VIA-0.6mm, F.Cu at (92.7, 118.7)
- added REF**: VIA-0.6mm, VIA-0.6mm, F.Cu at (122.9, 145.2)
- added REF**: VIA-0.6mm, VIA-0.6mm, F.Cu at (271.4, 99.4)
- added REF**: VIA-0.6mm, VIA-0.6mm, F.Cu at (315.1, 106.3)
- added REF**: VIA-0.6mm, VIA-0.6mm, F.Cu at (59.6, 99.1)
- added REF**: VIA-0.6mm, VIA-0.6mm, F.Cu at (106.8, 134.6)
- added REF**: VIA-0.6mm, VIA-0.6mm, F.Cu at (140.6, 152.3)
- added REF**: VIA-0.6mm, VIA-0.6mm, F.Cu at (45.4, 134.4)
- added REF**: VIA-0.6mm, VIA-0.6mm, F.Cu at (299.7, 118.7)
- added REF**: VIA-0.6mm, VIA-0.6mm, F.Cu at (52.5, 116.8)
- added REF**: VIA-0.6mm, VIA-0.6mm, F.Cu at (137.2, 110.0)
- added REF**: VIA-0.6mm, VIA-0.6mm, F.Cu at (99.8, 101.0)
- added REF**: VIA-0.6mm, VIA-0.6mm, F.Cu at (347.0, 134.4)
- added REF**: VIA-0.6mm, VIA-0.6mm, F.Cu at (255.2, 110.0)
- added _87: , Mount_Hole_2.2mm_Pad_Via, F.Cu at (185.7, 104.8)
- added _88: , Mount_Hole_2.2mm_Pad_Via, F.Cu at (206.7, 104.8)
- added _89: , Mount_Hole_2.2mm_Pad_Via, F.Cu at (185.7, 176.8)
- added _90: , Mount_Hole_2.2mm_Pad_Via, F.Cu at (206.7, 176.8)
- added _91: , Mount_Hole_2.2mm_Pad_Via, F.Cu at (176.1, 122.7)
- added _92: , Mount_Hole_2.2mm_Pad_Via, F.Cu at (175.9, 184.0)
- added _93: , Mount_Hole_2.2mm_Pad_Via, F.Cu at (96.9, 90.6)
- added _94: , Mount_Hole_2.2mm_Pad_Via, F.Cu at (106.9, 141.8)
- added _95: , Mount_Hole_2.2mm_Pad_Via, F.Cu at (216.2, 122.7)
- added _96: , Mount_Hole_2.2mm_Pad_Via, F.Cu at (216.4, 184.0)
- added _97: , Mount_Hole_2.2mm_Pad_Via, F.Cu at (295.5, 90.6)
- added _98: , Mount_Hole_2.2mm_Pad_Via, F.Cu at (285.4, 141.8)
- D1, D10, D11, D12, D13, D14, D15, D16, D17, D18, D19, D2, D20, D21, D22, D23, D24, D25, D26, D27, D28, D29, D3, D30, D31, D32, D33, D34, D35, D36, D37, D38, D39, D4, D40, D41, D42, D5, D6, D7, D8, D9: footprint Diode_SMD:D_SOD-323_HandSoldering -> Diode_SMD:D_SOD-323; moved to F.Cu
- MCU1: value Seeeduino XIAO-nrf52840 -> (none); footprint Seeeduino XIAO-MOUDLE14P-2.54-21X17.8MM -> ProMicro
- S1, S10, S11, S12, S13, S14, S15, S16, S17, S18, S19, S2, S20, S21, S22, S23, S24, S25, S26, S27, S28, S29, S3, S30, S31, S32, S33, S34, S35, S36, S37, S38, S39, S4, S40, S41, S42, S5, S6, S7, S8, S9: value Kailh-PG1425-X-Switch -> SW_MX_Choc_PCB_1.00u; footprint Kailh-PG1425-X-Switch -> SW_Cherry_MX_Choc_PCB_1.00u
- moved MCU1 112.8 mm to (196.2, 125.8), turned to -90 degrees
- moved D39 88.3 mm to (216.1, 110.6), turned to -68 degrees
- moved S21 87.2 mm to (164.5, 174.3), turned to -22 degrees
- moved S39 85.6 mm to (227.7, 112.9), turned to 22 degrees
- moved D36 83.8 mm to (233.8, 103.4), turned to -68 degrees
- moved D38 83.0 mm to (223.3, 128.2), turned to -68 degrees
- moved S42 81.2 mm to (227.9, 174.3), turned to 22 degrees
- moved S38 81.2 mm to (234.8, 130.5), turned to 22 degrees
- moved S20 81.2 mm to (146.9, 167.2), turned to -22 degrees
- moved D33 81.0 mm to (249.9, 92.8), turned to -68 degrees
- moved S36 80.3 mm to (245.3, 105.8), turned to 22 degrees
- moved D42 80.3 mm to (216.3, 172.0), turned to -68 degrees
- moved D35 78.3 mm to (240.9, 121.1), turned to -68 degrees
- moved D37 78.0 mm to (230.4, 145.8), turned to -68 degrees
- moved S37 77.1 mm to (241.9, 148.2), turned to 22 degrees
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Connections:
- D1 pad 1: P9 -> P104
- D10 pad 1: P9 -> P104
- D11 pad 1: P8 -> P106
- D12 pad 1: P7 -> P010
- D13 pad 1: P9 -> P104
- D14 pad 1: P8 -> P106
- D15 pad 1: P7 -> P010
- D16 pad 1: P9 -> P104
- D17 pad 1: P8 -> P106
- D18 pad 1: P7 -> P010
- D19 pad 1: P6 -> P009
- D2 pad 1: P8 -> P106
- D20 pad 1: P6 -> P009
- D21 pad 1: P6 -> P009
- D22 pad 1: P9_mirror -> P104
- D23 pad 1: P8_mirror -> P106
- D24 pad 1: P7_mirror -> P010
- D25 pad 1: P9_mirror -> P104
- D26 pad 1: P8_mirror -> P106
- D27 pad 1: P7_mirror -> P010
- D28 pad 1: P9_mirror -> P104
- D29 pad 1: P8_mirror -> P106
- D3 pad 1: P7 -> P010
- D30 pad 1: P7_mirror -> P010
- D31 pad 1: P9_mirror -> P104
- D32 pad 1: P8_mirror -> P106
- D33 pad 1: P7_mirror -> P010
- D34 pad 1: P9_mirror -> P104
- D35 pad 1: P8_mirror -> P106
- D36 pad 1: P7_mirror -> P010
- D37 pad 1: P9_mirror -> P104
- D38 pad 1: P8_mirror -> P106
- D39 pad 1: P7_mirror -> P010
- D4 pad 1: P9 -> P104
- D40 pad 1: P6_mirror -> P009
- D41 pad 1: P6_mirror -> P009
- D42 pad 1: P6_mirror -> P009
- D5 pad 1: P8 -> P106
- D6 pad 1: P7 -> P010
- D7 pad 1: P9 -> P104
- D8 pad 1: P8 -> P106
- D9 pad 1: P7 -> P010
- MCU1 pad 1: P0 -> RAW
- MCU1 pad 10: P9 -> P113
- MCU1 pad 11: P10 -> P111
- MCU1 pad 12: VCC -> P010
- MCU1 pad 13: GND -> P009
- MCU1 pad 14: RAW -> GND
- MCU1 pad 17: (no net) -> GND
- MCU1 pad 18: (no net) -> GND
- MCU1 pad 19: (no net) -> P017
- MCU1 pad 2: P1 -> RAW
- MCU1 pad 20: (no net) -> P020
- MCU1 pad 3: P2 -> GND
- MCU1 pad 4: P3 -> RST
- MCU1 pad 5: P4 -> VCC
- MCU1 pad 6: P5 -> P031
- MCU1 pad 7: P6 -> P029
- MCU1 pad 8: P7 -> P002
- MCU1 pad 9: P8 -> P115
- S1 pad 1: P0 -> P031
- S10 pad 1: P3 -> P115
- S11 pad 1: P3 -> P115
- S12 pad 1: P3 -> P115
- S13 pad 1: P4 -> P113
- S14 pad 1: P4 -> P113
- S15 pad 1: P4 -> P113
- S16 pad 1: P5 -> P111
- S17 pad 1: P5 -> P111
- S18 pad 1: P5 -> P111
- S19 pad 1: P3 -> P115
- S2 pad 1: P0 -> P031
- S20 pad 1: P4 -> P113
- S21 pad 1: P5 -> P111
- S22 pad 1: P0_mirror -> P017
- S23 pad 1: P0_mirror -> P017
- S24 pad 1: P0_mirror -> P017
- S25 pad 1: P1_mirror -> P020
- S26 pad 1: P1_mirror -> P020
- S27 pad 1: P1_mirror -> P020
- S28 pad 1: P2_mirror -> P022
- S29 pad 1: P2_mirror -> P022
- S3 pad 1: P0 -> P031
- S30 pad 1: P2_mirror -> P022
- S31 pad 1: P3_mirror -> P024
- S32 pad 1: P3_mirror -> P024
- S33 pad 1: P3_mirror -> P024
- S34 pad 1: P4_mirror -> P100
- S35 pad 1: P4_mirror -> P100
- S36 pad 1: P4_mirror -> P100
- S37 pad 1: P5_mirror -> P011
- S38 pad 1: P5_mirror -> P011
- S39 pad 1: P5_mirror -> P011
- S4 pad 1: P1 -> P029
- S40 pad 1: P3_mirror -> P024
- S41 pad 1: P4_mirror -> P100
- S42 pad 1: P5_mirror -> P011
- S5 pad 1: P1 -> P029
- S6 pad 1: P1 -> P029
- S7 pad 1: P2 -> P002
- S8 pad 1: P2 -> P002
- S9 pad 1: P2 -> P002
Routing:
- net RAW: track 384.8 -> 0.00 mm
- net P6: track 202.8 -> 0.00 mm, vias 1 -> 0
- net P6_mirror: track 192.9 -> 0.00 mm, vias 1 -> 0
- net P9: track 183.2 -> 0.00 mm, vias 1 -> 0
- net P8: track 165.9 -> 0.00 mm, vias 1 -> 0
- net P5: track 162.6 -> 0.00 mm
- net P9_mirror: track 161.8 -> 0.00 mm, vias 1 -> 0
- net P5_mirror: track 159.6 -> 0.00 mm
- net P7: track 150.1 -> 0.00 mm, vias 1 -> 0
- net P4: track 144.0 -> 0.00 mm
- net P8_mirror: track 144.0 -> 0.00 mm, vias 1 -> 0
- net P4_mirror: track 143.7 -> 0.00 mm
- net BAT_VCC: track 139.5 -> 0.00 mm
- net P3: track 130.1 -> 0.00 mm
- net P3_mirror: track 128.2 -> 0.00 mm
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- removed copper zone on B.Cu, net GND
- removed copper zone on F.Cu, net GND
Other:
- board size 291.8 x 81 mm -> 311 x 111 mm
- board text added: "by @kumekay 2024"
- board text added: "crabapplepad v2.0"
- board text removed: "+5V"
- board text removed: "GND"
- board text removed: "crabapplepad v1.0 by @kumekay 2023 left side"
- board text removed: "crabapplepad v1.0 by @kumekay 2023 right side"

Commit message: feat: wip version of the board
Parts:
- moved ? 1.27 mm to (162.4, 155.3)
- moved ? 1.27 mm to (194.2, 145.1)
- moved ? 1.27 mm to (198.2, 145.1)
- moved ? 1.27 mm to (161.5, 157.6)
- moved ? 1.27 mm to (207.2, 143.6)
- moved ? 1.27 mm to (164.3, 150.5)
- moved ? 1.27 mm to (225.1, 143.5)
- moved ? 1.27 mm to (163.4, 152.9)
- moved ? 1.27 mm to (228.0, 150.5)
- moved ? 1.27 mm to (185.2, 133.4)
- moved ? 1.27 mm to (185.2, 141.0)
- moved ? 1.27 mm to (167.2, 143.5)
- moved ? 1.27 mm to (185.2, 143.6)
- moved ? 1.27 mm to (165.3, 148.2)
- moved ? 1.27 mm to (229.9, 155.3)
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Routing:
- net P010: track 0.00 -> 312.4 mm
- net P104: track 0.00 -> 210.5 mm, vias 0 -> 1
- net P017: track 0.00 -> 204.6 mm
- net P106: track 0.00 -> 201.6 mm
- net P009: track 0.00 -> 170.8 mm
- net P020: track 0.00 -> 167.2 mm
- net P024: track 0.00 -> 145.4 mm
- net P022: track 0.00 -> 133.3 mm
- net P100: track 0.00 -> 108.0 mm
- net P011: track 0.00 -> 83.7 mm
- net P115: track 0.00 -> 83.4 mm
- net P113: track 0.00 -> 81.4 mm
- net P111: track 0.00 -> 77.6 mm
- net RAW: track 0.00 -> 69.6 mm
- net P002: track 0.00 -> 51.6 mm
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