File: hw/pcbs/kbd.kicad_pcb (KiCad board)
At the start: 2 copper layers, 311 x 111 mm, 182 parts

Commit message: feat: v2 production files
Parts:
- removed the ? at (162.4, 155.3)
- removed the ? at (194.2, 145.1)
- removed the ? at (168.2, 141.1)
- removed the ? at (198.2, 145.1)
- removed the ? at (161.5, 157.6)
- removed the ? at (207.2, 143.6)
- removed the ? at (164.3, 150.5)
- removed the ? at (185.2, 138.5)
- removed the ? at (225.1, 143.5)
- removed the ? at (163.4, 152.9)
- removed the ? at (185.2, 146.1)
- removed the ? at (228.0, 150.5)
- removed the ? at (185.2, 133.4)
- removed the ? at (207.2, 130.9)
- removed the ? at (207.2, 125.8)
- removed the ? at (185.2, 125.8)
- removed the ? at (185.2, 141.0)
- removed the ? at (167.2, 143.5)
- removed the ? at (185.2, 123.3)
- removed the ? at (185.2, 143.6)
- removed the ? at (165.3, 148.2)
- removed the ? at (229.9, 155.3)
- removed the ? at (207.2, 128.3)
- removed the ? at (160.5, 160.0)
- removed the ? at (229.0, 152.9)
- removed the ? at (185.2, 136.0)
- removed the ? at (207.2, 123.3)
- removed the ? at (207.2, 138.5)
- removed the ? at (230.9, 157.6)
- removed the ? at (227.1, 148.2)
- removed the ? at (231.8, 160.0)
- removed the ? at (207.2, 146.1)
- removed the ? at (224.2, 141.1)
- removed the ? at (226.1, 145.8)
- removed the ? at (207.2, 136.0)
- removed the ? at (223.2, 138.8)
- removed the ? at (185.2, 128.3)
- removed the ? at (185.2, 130.9)
- removed the ? at (207.2, 141.0)
- removed the ? at (169.1, 138.8)
- removed the ? at (166.3, 145.8)
- removed the ? at (207.2, 133.4)
- removed the REF** at (251.8, 153.6)
- removed the REF** at (237.6, 118.4)
- removed the REF** at (137.0, 172.7)
- removed the REF** at (269.4, 146.5)
- removed the REF** at (85.6, 137.6)
- removed the REF** at (121.0, 100.6)
- removed the REF** at (119.4, 165.5)
- removed the REF** at (237.8, 179.8)
- removed the REF** at (113.9, 118.2)
- removed the REF** at (273.0, 165.5)
- removed the REF** at (63.0, 142.8)
- removed the REF** at (322.3, 125.1)
- removed the REF** at (244.7, 136.0)
- removed the REF** at (262.3, 128.9)
- removed the REF** at (332.8, 100.4)
- removed the REF** at (77.2, 107.5)
- removed the REF** at (255.4, 172.7)
- removed the REF** at (70.1, 125.1)
- removed the REF** at (285.6, 135.9)
- removed the REF** at (306.8, 137.6)
- removed the REF** at (329.4, 142.8)
- removed the REF** at (339.9, 118.0)
- removed the REF** at (292.5, 102.3)
- removed the REF** at (147.7, 136.0)
- removed the REF** at (154.8, 118.4)
- removed the REF** at (130.1, 128.9)
- removed the REF** at (154.6, 179.8)
- removed the REF** at (278.5, 118.2)
- removed the REF** at (92.7, 119.9)
- removed the REF** at (122.9, 146.5)
- removed the REF** at (271.4, 100.6)
- removed the REF** at (315.1, 107.5)
- removed the REF** at (59.6, 100.4)
- removed the REF** at (106.8, 135.9)
- removed the REF** at (140.6, 153.6)
- removed the REF** at (45.4, 135.6)
- removed the REF** at (299.7, 119.9)
- removed the REF** at (52.5, 118.0)
- removed the REF** at (137.2, 111.3)
- removed the REF** at (99.8, 102.3)
- removed the REF** at (347.0, 135.6)
- removed the REF** at (255.2, 111.3)
- removed _87, _88, _89, _90, _91, _92, _93, _94, _95, _96, _97, _98: , Mount_Hole_2.2mm_Pad_Via
- added ?: , PAD-1.0922mm, F.Cu at (233.1, 125.2)
- added ?: , PAD-1.0922mm, F.Cu at (225.1, 115.1)
- added ?: , PAD-1.0922mm, F.Cu at (233.1, 132.8)
- added ?: , PAD-1.0922mm, F.Cu at (203.1, 122.7)
- added ?: , PAD-1.0922mm, F.Cu at (225.1, 132.8)
- added ?: , PAD-1.0922mm, F.Cu at (195.1, 120.1)
- added ?: , PAD-1.0922mm, F.Cu at (216.1, 128.7)
- added ?: , PAD-1.0922mm, F.Cu at (195.1, 110.0)
- added ?: , PAD-1.0922mm, F.Cu at (233.1, 117.6)
- added ?: , PAD-1.0922mm, F.Cu at (225.1, 127.8)
- added ?: , PAD-1.0922mm, F.Cu at (233.1, 112.5)
- added ?: , PAD-1.0922mm, F.Cu at (233.1, 110.0)
- added ?: , PAD-1.0922mm, F.Cu at (195.1, 130.3)
- added ?: , PAD-1.0922mm, F.Cu at (203.1, 125.2)
- added ?: , PAD-1.0922mm, F.Cu at (225.1, 130.3)
- added ?: , PAD-1.0922mm, F.Cu at (203.1, 112.5)
- added ?: , PAD-1.0922mm, F.Cu at (225.1, 112.5)
- added ?: , PAD-1.0922mm, F.Cu at (195.1, 112.5)
- added ?: , PAD-1.0922mm, F.Cu at (203.1, 130.3)
- added ?: , PAD-1.0922mm, F.Cu at (233.1, 120.1)
- added ?: , PAD-1.0922mm, F.Cu at (203.1, 127.8)
- added ?: , PAD-1.0922mm, F.Cu at (195.1, 115.1)
- added ?: , PAD-1.0922mm, F.Cu at (203.1, 115.1)
- added ?: , PAD-1.0922mm, F.Cu at (203.1, 132.8)
- added ?: , PAD-1.0922mm, F.Cu at (225.1, 125.2)
- added ?: , PAD-1.0922mm, F.Cu at (233.1, 122.7)
- added ?: , PAD-1.0922mm, F.Cu at (225.1, 122.7)
- added ?: , PAD-1.0922mm, F.Cu at (225.1, 117.6)
- added ?: , PAD-1.0922mm, F.Cu at (233.1, 115.1)
- added ?: , PAD-1.0922mm, F.Cu at (203.1, 117.6)
- added ?: , PAD-1.0922mm, F.Cu at (195.1, 132.8)
- added ?: , PAD-1.0922mm, F.Cu at (212.1, 128.7)
- added ?: , PAD-1.0922mm, F.Cu at (195.1, 122.7)
- added ?: , PAD-1.0922mm, F.Cu at (203.1, 120.1)
- added ?: , PAD-1.0922mm, F.Cu at (225.1, 120.1)
- added ?: , PAD-1.0922mm, F.Cu at (195.1, 127.8)
- added ?: , PAD-1.0922mm, F.Cu at (195.1, 125.2)
- added ?: , PAD-1.0922mm, F.Cu at (233.1, 130.3)
- added ?: , PAD-1.0922mm, F.Cu at (203.1, 110.0)
- added ?: , PAD-1.0922mm, F.Cu at (195.1, 117.6)
- added ?: , PAD-1.0922mm, F.Cu at (233.1, 127.8)
- added ?: , PAD-1.0922mm, F.Cu at (225.1, 110.0)
- added REF**: VIA-0.6mm, VIA-0.6mm, F.Cu at (116.5, 84.1)
- added REF**: VIA-0.6mm, VIA-0.6mm, F.Cu at (306.9, 77.2)
- added REF**: VIA-0.6mm, VIA-0.6mm, F.Cu at (84.6, 112.2)
- added REF**: VIA-0.6mm, VIA-0.6mm, F.Cu at (160.3, 77.2)
- added REF**: VIA-0.6mm, VIA-0.6mm, F.Cu at (158.5, 147.5)
- added REF**: VIA-0.6mm, VIA-0.6mm, F.Cu at (252.2, 154.6)
- added REF**: VIA-0.6mm, VIA-0.6mm, F.Cu at (268.0, 77.2)
- added REF**: VIA-0.6mm, VIA-0.6mm, F.Cu at (329.5, 82.4)
- added REF**: VIA-0.6mm, VIA-0.6mm, F.Cu at (84.5, 117.6)
- added REF**: VIA-0.6mm, VIA-0.6mm, F.Cu at (142.5, 75.5)
- added REF**: VIA-0.6mm, VIA-0.6mm, F.Cu at (132.0, 96.5)
- added REF**: VIA-0.6mm, VIA-0.6mm, F.Cu at (176.2, 149.2)
- added REF**: VIA-0.6mm, VIA-0.6mm, F.Cu at (318.9, 101.7)
- added REF**: VIA-0.6mm, VIA-0.6mm, F.Cu at (289.2, 78.9)
- added REF**: VIA-0.6mm, VIA-0.6mm, F.Cu at (98.7, 82.4)
- added REF**: VIA-0.6mm, VIA-0.6mm, F.Cu at (361.4, 110.5)
- added REF**: VIA-0.6mm, VIA-0.6mm, F.Cu at (102.3, 119.3)
- added REF**: VIA-0.6mm, VIA-0.6mm, F.Cu at (128.3, 110.7)
- added REF**: VIA-0.6mm, VIA-0.6mm, F.Cu at (292.9, 93.1)
- added REF**: VIA-0.6mm, VIA-0.6mm, F.Cu at (74.0, 92.9)
- added REF**: VIA-0.6mm, VIA-0.6mm, F.Cu at (241.3, 112.5)
- added REF**: VIA-0.6mm, VIA-0.6mm, F.Cu at (140.9, 140.4)
- added REF**: VIA-0.6mm, VIA-0.6mm, F.Cu at (258.9, 105.4)
- added REF**: VIA-0.6mm, VIA-0.6mm, F.Cu at (347.1, 75.3)
- added REF**: VIA-0.6mm, VIA-0.6mm, F.Cu at (194.1, 94.9)
- added REF**: VIA-0.6mm, VIA-0.6mm, F.Cu at (66.9, 110.5)
- added REF**: VIA-0.6mm, VIA-0.6mm, F.Cu at (187.0, 112.5)
- added REF**: VIA-0.6mm, VIA-0.6mm, F.Cu at (153.1, 94.8)
- added REF**: VIA-0.6mm, VIA-0.6mm, F.Cu at (146.0, 112.4)
- added REF**: VIA-0.6mm, VIA-0.6mm, F.Cu at (343.8, 117.6)
- added REF**: VIA-0.6mm, VIA-0.6mm, F.Cu at (303.4, 114.1)
- added REF**: VIA-0.6mm, VIA-0.6mm, F.Cu at (234.4, 156.3)
- added REF**: VIA-0.6mm, VIA-0.6mm, F.Cu at (179.8, 130.2)
- added REF**: VIA-0.6mm, VIA-0.6mm, F.Cu at (176.5, 87.8)
- added REF**: VIA-0.6mm, VIA-0.6mm, F.Cu at (266.0, 123.0)
- added REF**: VIA-0.6mm, VIA-0.6mm, F.Cu at (109.4, 101.7)
- added REF**: VIA-0.6mm, VIA-0.6mm, F.Cu at (144.5, 121.4)
- added REF**: VIA-0.6mm, VIA-0.6mm, F.Cu at (124.9, 114.1)
- added REF**: VIA-0.6mm, VIA-0.6mm, F.Cu at (114.2, 94.8)
- added REF**: VIA-0.6mm, VIA-0.6mm, F.Cu at (343.6, 112.2)
- added REF**: VIA-0.6mm, VIA-0.6mm, F.Cu at (321.2, 112.4)
- added REF**: VIA-0.6mm, VIA-0.6mm, F.Cu at (259.1, 110.9)
- added REF**: VIA-0.6mm, VIA-0.6mm, F.Cu at (311.8, 84.1)
- added REF**: VIA-0.6mm, VIA-0.6mm, F.Cu at (135.4, 93.1)
- added REF**: VIA-0.6mm, VIA-0.6mm, F.Cu at (151.6, 103.8)
- added REF**: VIA-0.6mm, VIA-0.6mm, F.Cu at (285.7, 75.5)
- added REF**: VIA-0.6mm, VIA-0.6mm, F.Cu at (162.2, 123.0)
- added REF**: VIA-0.6mm, VIA-0.6mm, F.Cu at (91.6, 100.0)
- added REF**: VIA-0.6mm, VIA-0.6mm, F.Cu at (269.6, 86.1)
- added REF**: VIA-0.6mm, VIA-0.6mm, F.Cu at (336.5, 94.6)
- added REF**: VIA-0.6mm, VIA-0.6mm, F.Cu at (266.2, 128.5)
- added REF**: VIA-0.6mm, VIA-0.6mm, F.Cu at (248.4, 130.2)
- added REF**: VIA-0.6mm, VIA-0.6mm, F.Cu at (283.8, 121.4)
- added REF**: VIA-0.6mm, VIA-0.6mm, F.Cu at (336.6, 100.0)
- added REF**: VIA-0.6mm, VIA-0.6mm, F.Cu at (158.6, 142.1)
- added REF**: VIA-0.6mm, VIA-0.6mm, F.Cu at (275.1, 94.8)
- added REF**: VIA-0.6mm, VIA-0.6mm, F.Cu at (287.4, 140.4)
- added REF**: VIA-0.6mm, VIA-0.6mm, F.Cu at (269.6, 142.1)
- added REF**: VIA-0.6mm, VIA-0.6mm, F.Cu at (176.1, 154.6)
- added REF**: VIA-0.6mm, VIA-0.6mm, F.Cu at (251.8, 87.8)
- added REF**: VIA-0.6mm, VIA-0.6mm, F.Cu at (314.0, 94.8)
- added REF**: VIA-0.6mm, VIA-0.6mm, F.Cu at (296.3, 96.5)
- added REF**: VIA-0.6mm, VIA-0.6mm, F.Cu at (276.7, 103.8)
- added REF**: VIA-0.6mm, VIA-0.6mm, F.Cu at (139.1, 78.9)
- added REF**: VIA-0.6mm, VIA-0.6mm, F.Cu at (234.2, 94.9)
- added REF**: VIA-0.6mm, VIA-0.6mm, F.Cu at (81.1, 75.3)
- added REF**: VIA-0.6mm, VIA-0.6mm, F.Cu at (176.3, 93.3)
- added REF**: VIA-0.6mm, VIA-0.6mm, F.Cu at (252.0, 149.2)
- added REF**: VIA-0.6mm, VIA-0.6mm, F.Cu at (251.9, 93.3)
- added REF**: VIA-0.6mm, VIA-0.6mm, F.Cu at (354.3, 92.9)
- added REF**: VIA-0.6mm, VIA-0.6mm, F.Cu at (282.2, 112.4)
- added REF**: VIA-0.6mm, VIA-0.6mm, F.Cu at (329.4, 77.0)
- added REF**: VIA-0.6mm, VIA-0.6mm, F.Cu at (158.7, 86.1)
- added REF**: VIA-0.6mm, VIA-0.6mm, F.Cu at (193.9, 156.3)
- added REF**: VIA-0.6mm, VIA-0.6mm, F.Cu at (169.2, 110.9)
- added REF**: VIA-0.6mm, VIA-0.6mm, F.Cu at (162.1, 128.5)
- added REF**: VIA-0.6mm, VIA-0.6mm, F.Cu at (121.3, 77.2)
- added REF**: VIA-0.6mm, VIA-0.6mm, F.Cu at (300.0, 110.7)
- added REF**: VIA-0.6mm, VIA-0.6mm, F.Cu at (326.0, 119.3)
- added REF**: VIA-0.6mm, VIA-0.6mm, F.Cu at (91.8, 94.6)
- added REF**: VIA-0.6mm, VIA-0.6mm, F.Cu at (107.1, 112.4)
- added REF**: VIA-0.6mm, VIA-0.6mm, F.Cu at (98.9, 77.0)
- added REF**: VIA-0.6mm, VIA-0.6mm, F.Cu at (169.3, 105.4)
- added REF**: VIA-0.6mm, VIA-0.6mm, F.Cu at (269.8, 147.5)
- added _129: , Mount_Hole_2.2mm_Pad_Via, F.Cu at (203.6, 89.7)
- added _130: , Mount_Hole_2.2mm_Pad_Via, F.Cu at (224.6, 89.7)
- added _131: , Mount_Hole_2.2mm_Pad_Via, F.Cu at (203.6, 161.7)
- added _132: , Mount_Hole_2.2mm_Pad_Via, F.Cu at (224.6, 161.7)
- added _133: , Mount_Hole_2.2mm_Pad_Via, F.Cu at (191.7, 88.2)
- added _134: , Mount_Hole_2.2mm_Pad_Via, F.Cu at (193.9, 169.0)
- added _135: , Mount_Hole_2.2mm_Pad_Via, F.Cu at (114.8, 75.6)
- added _136: , Mount_Hole_2.2mm_Pad_Via, F.Cu at (124.9, 126.8)
- added _137: , Mount_Hole_2.2mm_Pad_Via, F.Cu at (236.6, 88.2)
- added _138: , Mount_Hole_2.2mm_Pad_Via, F.Cu at (234.4, 169.0)
- added _139: , Mount_Hole_2.2mm_Pad_Via, F.Cu at (313.4, 75.6)
- added _140: , Mount_Hole_2.2mm_Pad_Via, F.Cu at (303.4, 126.8)
- D1, D10, D11, D12, D13, D14, D15, D16, D17, D18, D19, D2, D20, D21, D22, D23, D24, D25, D26, D27, D28, D29, D3, D30, D31, D32, D33, D34, D35, D36, D37, D38, D39, D4, D40, D41, D42, D5, D6, D7, D8, D9: footprint Diode_SMD:D_SOD-323 -> Diode_SMD:D_SOD-323_HandSoldering
- moved S36 24.3 mm to (263.2, 90.7)
- moved S24 24.3 mm to (340.8, 79.9)
- moved S13 24.3 mm to (150.8, 126.0)
- moved S4 24.3 mm to (90.8, 122.2)
- moved MCU1 24.3 mm to (214.1, 110.7)
- moved S19 24.3 mm to (147.2, 145.0)
- moved S41 24.3 mm to (263.4, 152.1)
- moved S28 24.3 mm to (314.8, 117.0)
- moved S5 24.3 mm to (97.9, 104.6)
- moved S26 24.3 mm to (330.3, 104.6)
- moved S8 24.3 mm to (120.5, 99.4)
- moved S9 24.3 mm to (127.7, 81.8)
- moved S37 24.3 mm to (259.8, 133.1)
- moved S40 24.3 mm to (281.1, 145.0)
- moved S6 24.3 mm to (105.1, 87.0)
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Routing:
- net P031: track 50.1 -> 174.1 mm
- net P106: track 201.6 -> 323.9 mm, vias 0 -> 2
- net P104: track 210.5 -> 327.1 mm
- net P029: track 50.8 -> 143.9 mm
- net P002: track 51.6 -> 126.1 mm
- net P115: track 83.4 -> 136.0 mm
- net P017: track 204.6 -> 169.9 mm
- net P113: track 81.4 -> 115.5 mm, vias 0 -> 1
- net P020: track 167.2 -> 134.1 mm
- net P111: track 77.6 -> 98.8 mm
- net P022: track 133.3 -> 116.7 mm
- net P009: track 170.8 -> 186.2 mm, vias 0 -> 1
- net mirror_index_home: track 13.4 -> 0.00 mm
- net mirror_inner_home: track 13.4 -> 0.00 mm
- net mirror_ring_home: track 13.4 -> 0.00 mm
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- added copper zone on B.Cu, net GND
- added copper zone on F.Cu, net GND

Commit message: fix: Update production files
Parts:
- ? (x42): footprint PAD-1.0922mm -> SW_MX_Choc:PAD-1mm
- D1, D10, D11, D12, D13, D14, D15, D16, D17, D18, D19, D2, D20, D21, D22, D23, D24, D25, D26, D27, D28, D29, D3, D30, D31, D32, D33, D34, D35, D36, D37, D38, D39, D4, D40, D41, D42, D5, D6, D7, D8, D9: footprint Diode_SMD:D_SOD-323_HandSoldering -> SW_MX_Choc:D_SOD-323_HandSoldering
- S1, S10, S11, S12, S13, S14, S15, S16, S17, S18, S19, S2, S20, S21, S22, S23, S24, S25, S26, S27, S28, S29, S3, S30, S31, S32, S33, S34, S35, S36, S37, S38, S39, S4, S40, S41, S42, S5, S6, S7, S8, S9: footprint SW_Cherry_MX_Choc_PCB_1.00u -> SW_MX_Choc:SW_Cherry_MX_Choc_PCB_1.00u_nosilk
- _129, _130, _131, _132, _133, _134, _135, _136, _137, _138, _139, _140: footprint Mount_Hole_2.2mm_Pad_Via -> MountingHole:MountingHole_2.2mm_M2_DIN965
- moved ? 17.4 mm to (238.0, 149.6)
- moved PWR1 17.4 mm to (219.0, 180.2)
- moved REF** 17.4 mm to (163.4, 164.3)
- moved REF** 17.4 mm to (334.2, 93.7)
- moved ? 17.4 mm to (238.0, 142.0)
- moved ? 17.4 mm to (238.0, 139.4)
- moved D9 17.4 mm to (142.8, 98.4)
- moved REF** 17.4 mm to (256.8, 110.0)
- moved ? 17.4 mm to (238.0, 129.3)
- moved D38 17.4 mm to (247.3, 132.1)
- moved REF** 17.4 mm to (89.5, 128.9)
- moved REF** 17.4 mm to (294.0, 95.6)
- moved S25 17.4 mm to (342.3, 139.0)
- moved _140 17.4 mm to (308.3, 143.5)
- moved ? 17.4 mm to (230.0, 129.3)
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Routing:
- net P010: track 320.8 -> 353.5 mm, vias 1 -> 3
- net mirror_ring_home: track 0.00 -> 12.8 mm
- net mirror_middle_home: track 0.00 -> 12.8 mm
- net mirror_index_home: track 0.00 -> 12.8 mm
- net mirror_inner_home: track 0.00 -> 12.8 mm
- net GND: track 0.00 -> 11.0 mm, vias 7 -> 16
- net pinky_home: track 0.00 -> 7.73 mm
- net P115: track 136.0 -> 134.2 mm
- net RAW: track 68.5 -> 70.2 mm
- net P104: track 327.1 -> 325.4 mm
- net P024: track 145.1 -> 143.6 mm
- net P029: track 143.9 -> 142.4 mm
- net P031: track 174.1 -> 172.8 mm
- net P009: track 186.2 -> 184.9 mm
- net P106: track 323.9 -> 322.9 mm
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